Commit message: Add servo visual and collision meshes to URDF; update joint origins and inertial properties for improved accuracy

File: hexapod-v2/hexapod-v2.urdf (robot description, URDF)
Before this commit: robot hexapod_v2, 25 links, 24 joints
Links:
- link l1_coxa: geometry collision mesh filename=package://hexapod_v2/coxa-996-left.stl scale=0.001 0.001 0.001; collision mesh filename=package://hexapod_v2/servo-MG996R.stl scale=0.001 0.001 0.001
- link l1_femur: geometry collision mesh filename=package://hexapod_v2/femur-996-left.stl scale=0.001 0.001 0.001; collision mesh filename=package://hexapod_v2/servo-MG996R.stl scale=0.001 0.001 0.001
- link l1_tibia: geometry collision mesh filename=package://hexapod_v2/servo-MG996R.stl scale=0.001 0.001 0.001; collision mesh filename=package://hexapod_v2/tibia-996-left.stl scale=0.001 0.001 0.001
- link l2_coxa: geometry collision mesh filename=package://hexapod_v2/coxa-996-left.stl scale=0.001 0.001 0.001; collision mesh filename=package://hexapod_v2/servo-MG996R.stl scale=0.001 0.001 0.001
- link l2_femur: geometry collision mesh filename=package://hexapod_v2/femur-996-left.stl scale=0.001 0.001 0.001; collision mesh filename=package://hexapod_v2/servo-MG996R.stl scale=0.001 0.001 0.001
- link l2_tibia: geometry collision mesh filename=package://hexapod_v2/servo-MG996R.stl scale=0.001 0.001 0.001; collision mesh filename=package://hexapod_v2/tibia-996-left.stl scale=0.001 0.001 0.001
- link l3_coxa: geometry collision mesh filename=package://hexapod_v2/coxa-996-left.stl scale=0.001 0.001 0.001; collision mesh filename=package://hexapod_v2/servo-MG996R.stl scale=0.001 0.001 0.001
- link l3_femur: geometry collision mesh filename=package://hexapod_v2/femur-996-left.stl scale=0.001 0.001 0.001; collision mesh filename=package://hexapod_v2/servo-MG996R.stl scale=0.001 0.001 0.001
- link l3_tibia: geometry collision mesh filename=package://hexapod_v2/servo-MG996R.stl scale=0.001 0.001 0.001; collision mesh filename=package://hexapod_v2/tibia-996-left.stl scale=0.001 0.001 0.001
- link r1_coxa: geometry collision mesh filename=package://hexapod_v2/coxa-996-right.stl scale=0.001 0.001 0.001; collision mesh filename=package://hexapod_v2/servo-MG996R.stl scale=0.001 0.001 0.001
- link r1_femur: geometry collision mesh filename=package://hexapod_v2/femur-996-right.stl scale=0.001 0.001 0.001; collision mesh filename=package://hexapod_v2/servo-MG996R.stl scale=0.001 0.001 0.001
- link r1_tibia: geometry collision mesh filename=package://hexapod_v2/servo-MG996R.stl scale=0.001 0.001 0.001; collision mesh filename=package://hexapod_v2/tibia-996-right.stl scale=0.001 0.001 0.001
- link r2_coxa: geometry collision mesh filename=package://hexapod_v2/coxa-996-right.stl scale=0.001 0.001 0.001; collision mesh filename=package://hexapod_v2/servo-MG996R.stl scale=0.001 0.001 0.001
- link r2_femur: geometry collision mesh filename=package://hexapod_v2/femur-996-right.stl scale=0.001 0.001 0.001; collision mesh filename=package://hexapod_v2/servo-MG996R.stl scale=0.001 0.001 0.001
- link r2_tibia: geometry collision mesh filename=package://hexapod_v2/servo-MG996R.stl scale=0.001 0.001 0.001; collision mesh filename=package://hexapod_v2/tibia-996-right.stl scale=0.001 0.001 0.001
- link r3_coxa: geometry collision mesh filename=package://hexapod_v2/coxa-996-right.stl scale=0.001 0.001 0.001; collision mesh filename=package://hexapod_v2/servo-MG996R.stl scale=0.001 0.001 0.001
- link r3_femur: geometry collision mesh filename=package://hexapod_v2/femur-996-right.stl scale=0.001 0.001 0.001; collision mesh filename=package://hexapod_v2/servo-MG996R.stl scale=0.001 0.001 0.001
- link r3_tibia: geometry collision mesh filename=package://hexapod_v2/servo-MG996R.stl scale=0.001 0.001 0.001; collision mesh filename=package://hexapod_v2/tibia-996-right.stl scale=0.001 0.001 0.001
Joints:
- joint l1_tip_joint: origin xyz=0.134000 0.000000 0.000000 rpy=0.000000 0.000000 0.000000 -> xyz=0.100076 0.000000 0.000000 rpy=0.000000 0.000000 0.000000
- joint l2_tip_joint: origin xyz=0.134000 0.000000 0.000000 rpy=0.000000 0.000000 0.000000 -> xyz=0.100076 0.000000 0.000000 rpy=0.000000 0.000000 0.000000
- joint l3_tip_joint: origin xyz=0.134000 0.000000 0.000000 rpy=0.000000 0.000000 0.000000 -> xyz=0.100076 0.000000 0.000000 rpy=0.000000 0.000000 0.000000
- joint r1_tip_joint: origin xyz=0.134000 0.000000 0.000000 rpy=0.000000 0.000000 0.000000 -> xyz=0.100076 0.000000 0.000000 rpy=0.000000 0.000000 0.000000
- joint r2_tip_joint: origin xyz=0.134000 0.000000 0.000000 rpy=0.000000 0.000000 0.000000 -> xyz=0.100076 0.000000 0.000000 rpy=0.000000 0.000000 0.000000
- joint r3_tip_joint: origin xyz=0.134000 0.000000 0.000000 rpy=0.000000 0.000000 0.000000 -> xyz=0.100076 0.000000 0.000000 rpy=0.000000 0.000000 0.000000

Commit message: Update mesh file paths in URDF to use relative paths for improved compatibility with viewers

File: hexapod-v2/hexapod-v2.urdf (robot description, URDF)
Before this commit: robot hexapod_v2, 25 links, 24 joints
Links:
- link base_link: geometry collision mesh filename=./frame.stl scale=0.001 0.001 0.001; collision mesh filename=./servo2040-bottom-cover (a).stl scale=0.001 0.001 0.001
- link l1_coxa: geometry collision mesh filename=./coxa-996-left.stl scale=0.001 0.001 0.001; collision mesh filename=./servo-MG996R.stl scale=0.001 0.001 0.001
- link l1_femur: geometry collision mesh filename=./femur-996-left.stl scale=0.001 0.001 0.001; collision mesh filename=./servo-MG996R.stl scale=0.001 0.001 0.001
- link l1_tibia: geometry collision mesh filename=./servo-MG996R.stl scale=0.001 0.001 0.001; collision mesh filename=./tibia-996-left.stl scale=0.001 0.001 0.001
- link l2_coxa: geometry collision mesh filename=./coxa-996-left.stl scale=0.001 0.001 0.001; collision mesh filename=./servo-MG996R.stl scale=0.001 0.001 0.001
- link l2_femur: geometry collision mesh filename=./femur-996-left.stl scale=0.001 0.001 0.001; collision mesh filename=./servo-MG996R.stl scale=0.001 0.001 0.001
- link l2_tibia: geometry collision mesh filename=./servo-MG996R.stl scale=0.001 0.001 0.001; collision mesh filename=./tibia-996-left.stl scale=0.001 0.001 0.001
- link l3_coxa: geometry collision mesh filename=./coxa-996-left.stl scale=0.001 0.001 0.001; collision mesh filename=./servo-MG996R.stl scale=0.001 0.001 0.001
- link l3_femur: geometry collision mesh filename=./femur-996-left.stl scale=0.001 0.001 0.001; collision mesh filename=./servo-MG996R.stl scale=0.001 0.001 0.001
- link l3_tibia: geometry collision mesh filename=./servo-MG996R.stl scale=0.001 0.001 0.001; collision mesh filename=./tibia-996-left.stl scale=0.001 0.001 0.001
- link r1_coxa: geometry collision mesh filename=./coxa-996-right.stl scale=0.001 0.001 0.001; collision mesh filename=./servo-MG996R.stl scale=0.001 0.001 0.001
- link r1_femur: geometry collision mesh filename=./femur-996-right.stl scale=0.001 0.001 0.001; collision mesh filename=./servo-MG996R.stl scale=0.001 0.001 0.001
- link r1_tibia: geometry collision mesh filename=./servo-MG996R.stl scale=0.001 0.001 0.001; collision mesh filename=./tibia-996-right.stl scale=0.001 0.001 0.001
- link r2_coxa: geometry collision mesh filename=./coxa-996-right.stl scale=0.001 0.001 0.001; collision mesh filename=./servo-MG996R.stl scale=0.001 0.001 0.001
- link r2_femur: geometry collision mesh filename=./femur-996-right.stl scale=0.001 0.001 0.001; collision mesh filename=./servo-MG996R.stl scale=0.001 0.001 0.001
- link r2_tibia: geometry collision mesh filename=./servo-MG996R.stl scale=0.001 0.001 0.001; collision mesh filename=./tibia-996-right.stl scale=0.001 0.001 0.001
- link r3_coxa: geometry collision mesh filename=./coxa-996-right.stl scale=0.001 0.001 0.001; collision mesh filename=./servo-MG996R.stl scale=0.001 0.001 0.001
- link r3_femur: geometry collision mesh filename=./femur-996-right.stl scale=0.001 0.001 0.001; collision mesh filename=./servo-MG996R.stl scale=0.001 0.001 0.001
- link r3_tibia: geometry collision mesh filename=./servo-MG996R.stl scale=0.001 0.001 0.001; collision mesh filename=./tibia-996-right.stl scale=0.001 0.001 0.001

Commit message: Add servo links and joints for hexapod legs L1, L2, L3, R1, R2, R3
- Introduced new servo links (l1_hip_servo, l1_shoulder_servo, l1_knee_servo, etc.) for each leg.
- Updated visual and collision properties for the new servo links.
- Added fixed joints for each servo link to connect them to their respective parent links.
- Adjusted positions and orientations of existing links and joints to accommodate the new structure.
- Ensured consistent mass and inertia values across all servo links.

File: hexapod-v2/hexapod-v2.urdf (robot description, URDF)
Before this commit: robot hexapod_v2, 25 links, 24 joints
Links:
- added link l1_hip_servo, mass 0.055; collision mesh filename=./servo-MG996R.stl scale=0.001 0.001 0.001; visual mesh filename=./servo-MG996R.stl scale=0.001 0.001 0.001
- added link l1_knee_servo, mass 0.055; collision mesh filename=./servo-MG996R.stl scale=0.001 0.001 0.001; visual mesh filename=./servo-MG996R.stl scale=0.001 0.001 0.001
- added link l1_shoulder_servo, mass 0.055; collision mesh filename=./servo-MG996R.stl scale=0.001 0.001 0.001; visual mesh filename=./servo-MG996R.stl scale=0.001 0.001 0.001
- added link l2_hip_servo, mass 0.055; collision mesh filename=./servo-MG996R.stl scale=0.001 0.001 0.001; visual mesh filename=./servo-MG996R.stl scale=0.001 0.001 0.001
- added link l2_knee_servo, mass 0.055; collision mesh filename=./servo-MG996R.stl scale=0.001 0.001 0.001; visual mesh filename=./servo-MG996R.stl scale=0.001 0.001 0.001
- added link l2_shoulder_servo, mass 0.055; collision mesh filename=./servo-MG996R.stl scale=0.001 0.001 0.001; visual mesh filename=./servo-MG996R.stl scale=0.001 0.001 0.001
- added link l3_hip_servo, mass 0.055; collision mesh filename=./servo-MG996R.stl scale=0.001 0.001 0.001; visual mesh filename=./servo-MG996R.stl scale=0.001 0.001 0.001
- added link l3_knee_servo, mass 0.055; collision mesh filename=./servo-MG996R.stl scale=0.001 0.001 0.001; visual mesh filename=./servo-MG996R.stl scale=0.001 0.001 0.001
- added link l3_shoulder_servo, mass 0.055; collision mesh filename=./servo-MG996R.stl scale=0.001 0.001 0.001; visual mesh filename=./servo-MG996R.stl scale=0.001 0.001 0.001
- added link r1_hip_servo, mass 0.055; collision mesh filename=./servo-MG996R.stl scale=0.001 0.001 0.001; visual mesh filename=./servo-MG996R.stl scale=0.001 0.001 0.001
- added link r1_knee_servo, mass 0.055; collision mesh filename=./servo-MG996R.stl scale=0.001 0.001 0.001; visual mesh filename=./servo-MG996R.stl scale=0.001 0.001 0.001
- added link r1_shoulder_servo, mass 0.055; collision mesh filename=./servo-MG996R.stl scale=0.001 0.001 0.001; visual mesh filename=./servo-MG996R.stl scale=0.001 0.001 0.001
- added link r2_hip_servo, mass 0.055; collision mesh filename=./servo-MG996R.stl scale=0.001 0.001 0.001; visual mesh filename=./servo-MG996R.stl scale=0.001 0.001 0.001
- added link r2_knee_servo, mass 0.055; collision mesh filename=./servo-MG996R.stl scale=0.001 0.001 0.001; visual mesh filename=./servo-MG996R.stl scale=0.001 0.001 0.001
- added link r2_shoulder_servo, mass 0.055; collision mesh filename=./servo-MG996R.stl scale=0.001 0.001 0.001; visual mesh filename=./servo-MG996R.stl scale=0.001 0.001 0.001
- added link r3_hip_servo, mass 0.055; collision mesh filename=./servo-MG996R.stl scale=0.001 0.001 0.001; visual mesh filename=./servo-MG996R.stl scale=0.001 0.001 0.001
- added link r3_knee_servo, mass 0.055; collision mesh filename=./servo-MG996R.stl scale=0.001 0.001 0.001; visual mesh filename=./servo-MG996R.stl scale=0.001 0.001 0.001
- added link r3_shoulder_servo, mass 0.055; collision mesh filename=./servo-MG996R.stl scale=0.001 0.001 0.001; visual mesh filename=./servo-MG996R.stl scale=0.001 0.001 0.001
- link l1_coxa: geometry collision mesh filename=./coxa-996-left.stl scale=0.001 0.001 0.001; visual mesh filename=./coxa-996-left.stl scale=0.001 0.001 0.001
- link l1_femur: geometry collision mesh filename=./femur-996-left.stl scale=0.001 0.001 0.001; visual mesh filename=./femur-996-left.stl scale=0.001 0.001 0.001
- link l1_tibia: geometry collision mesh filename=./tibia-996-left.stl scale=0.001 0.001 0.001; visual mesh filename=./tibia-996-left.stl scale=0.001 0.001 0.001
- link l2_coxa: geometry collision mesh filename=./coxa-996-left.stl scale=0.001 0.001 0.001; visual mesh filename=./coxa-996-left.stl scale=0.001 0.001 0.001
- link l2_femur: geometry collision mesh filename=./femur-996-left.stl scale=0.001 0.001 0.001; visual mesh filename=./femur-996-left.stl scale=0.001 0.001 0.001
- link l2_tibia: geometry collision mesh filename=./tibia-996-left.stl scale=0.001 0.001 0.001; visual mesh filename=./tibia-996-left.stl scale=0.001 0.001 0.001
- link l3_coxa: geometry collision mesh filename=./coxa-996-left.stl scale=0.001 0.001 0.001; visual mesh filename=./coxa-996-left.stl scale=0.001 0.001 0.001
- link l3_femur: geometry collision mesh filename=./femur-996-left.stl scale=0.001 0.001 0.001; visual mesh filename=./femur-996-left.stl scale=0.001 0.001 0.001
- link l3_tibia: geometry collision mesh filename=./tibia-996-left.stl scale=0.001 0.001 0.001; visual mesh filename=./tibia-996-left.stl scale=0.001 0.001 0.001
- link r1_coxa: geometry collision mesh filename=./coxa-996-right.stl scale=0.001 0.001 0.001; visual mesh filename=./coxa-996-right.stl scale=0.001 0.001 0.001
- link r1_femur: geometry collision mesh filename=./femur-996-right.stl scale=0.001 0.001 0.001; visual mesh filename=./femur-996-right.stl scale=0.001 0.001 0.001
- link r1_tibia: geometry collision mesh filename=./tibia-996-right.stl scale=0.001 0.001 0.001; visual mesh filename=./tibia-996-right.stl scale=0.001 0.001 0.001
- link r2_coxa: geometry collision mesh filename=./coxa-996-right.stl scale=0.001 0.001 0.001; visual mesh filename=./coxa-996-right.stl scale=0.001 0.001 0.001
- link r2_femur: geometry collision mesh filename=./femur-996-right.stl scale=0.001 0.001 0.001; visual mesh filename=./femur-996-right.stl scale=0.001 0.001 0.001
- link r2_tibia: geometry collision mesh filename=./tibia-996-right.stl scale=0.001 0.001 0.001; visual mesh filename=./tibia-996-right.stl scale=0.001 0.001 0.001
- link r3_coxa: geometry collision mesh filename=./coxa-996-right.stl scale=0.001 0.001 0.001; visual mesh filename=./coxa-996-right.stl scale=0.001 0.001 0.001
- link r3_femur: geometry collision mesh filename=./femur-996-right.stl scale=0.001 0.001 0.001; visual mesh filename=./femur-996-right.stl scale=0.001 0.001 0.001
- link r3_tibia: geometry collision mesh filename=./tibia-996-right.stl scale=0.001 0.001 0.001; visual mesh filename=./tibia-996-right.stl scale=0.001 0.001 0.001
Joints:
- added joint l1_hip_servo_joint: type fixed, parent base_link, child l1_hip_servo, origin xyz=-0.063000 0.083500 0.000000 rpy=0.000000 0.000000 2.217165
- added joint l1_knee_servo_joint: type fixed, parent l1_femur, child l1_knee_servo, origin xyz=0.080000 0.000000 0.000000 rpy=0.000000 0.000000 0.000000
- added joint l1_shoulder_servo_joint: type fixed, parent l1_coxa, child l1_shoulder_servo, origin xyz=0.043000 0.000000 0.000000 rpy=0.000000 0.000000 0.000000
- added joint l2_hip_servo_joint: type fixed, parent base_link, child l2_hip_servo, origin xyz=-0.081500 0.000000 0.000000 rpy=0.000000 0.000000 3.141593
- added joint l2_knee_servo_joint: type fixed, parent l2_femur, child l2_knee_servo, origin xyz=0.080000 0.000000 0.000000 rpy=0.000000 0.000000 0.000000
- added joint l2_shoulder_servo_joint: type fixed, parent l2_coxa, child l2_shoulder_servo, origin xyz=0.043000 0.000000 0.000000 rpy=0.000000 0.000000 0.000000
- added joint l3_hip_servo_joint: type fixed, parent base_link, child l3_hip_servo, origin xyz=-0.063000 -0.083500 0.000000 rpy=0.000000 0.000000 -2.217165
- added joint l3_knee_servo_joint: type fixed, parent l3_femur, child l3_knee_servo, origin xyz=0.080000 0.000000 0.000000 rpy=0.000000 0.000000 0.000000
- added joint l3_shoulder_servo_joint: type fixed, parent l3_coxa, child l3_shoulder_servo, origin xyz=0.043000 0.000000 0.000000 rpy=0.000000 0.000000 0.000000
- added joint r1_hip_servo_joint: type fixed, parent base_link, child r1_hip_servo, origin xyz=0.063000 0.083500 0.000000 rpy=0.000000 0.000000 0.924427
- added joint r1_knee_servo_joint: type fixed, parent r1_femur, child r1_knee_servo, origin xyz=0.080000 0.000000 0.000000 rpy=0.000000 0.000000 0.000000
- added joint r1_shoulder_servo_joint: type fixed, parent r1_coxa, child r1_shoulder_servo, origin xyz=0.043000 0.000000 0.000000 rpy=0.000000 0.000000 0.000000
- added joint r2_hip_servo_joint: type fixed, parent base_link, child r2_hip_servo, origin xyz=0.081500 0.000000 0.000000 rpy=0.000000 0.000000 0.000000
- added joint r2_knee_servo_joint: type fixed, parent r2_femur, child r2_knee_servo, origin xyz=0.080000 0.000000 0.000000 rpy=0.000000 0.000000 0.000000
- added joint r2_shoulder_servo_joint: type fixed, parent r2_coxa, child r2_shoulder_servo, origin xyz=0.043000 0.000000 0.000000 rpy=0.000000 0.000000 0.000000
- added joint r3_hip_servo_joint: type fixed, parent base_link, child r3_hip_servo, origin xyz=0.063000 -0.083500 0.000000 rpy=0.000000 0.000000 -0.924427
- added joint r3_knee_servo_joint: type fixed, parent r3_femur, child r3_knee_servo, origin xyz=0.080000 0.000000 0.000000 rpy=0.000000 0.000000 0.000000
- added joint r3_shoulder_servo_joint: type fixed, parent r3_coxa, child r3_shoulder_servo, origin xyz=0.043000 0.000000 0.000000 rpy=0.000000 0.000000 0.000000
