Commit message: Add new STL mesh files for hexapod components
- Added bottom cover (flat and standard)
- Added left and right coxa
- Added left and right femur
- Added frame
- Added servo components (hip, limb left, limb right)
- Added left and right tibia
- Added top cover

File: hexapod-v2/hexapod-v2.urdf (robot description, URDF)
Before this commit: robot hexapod_v2, 43 links, 42 joints
Links:
- link base_link: geometry collision mesh filename=./meshes/bottom-cover-flat.stl scale=0.001 0.001 0.001; collision mesh filename=./meshes/frame.stl scale=0.001 0.001 0.001
- link l1_coxa: geometry collision mesh filename=./meshes/coxa-left.stl scale=0.001 0.001 0.001; visual mesh filename=./meshes/coxa-left.stl scale=0.001 0.001 0.001
- link l1_femur: geometry collision mesh filename=./meshes/femur-left.stl scale=0.001 0.001 0.001; visual mesh filename=./meshes/femur-left.stl scale=0.001 0.001 0.001
- link l1_hip_servo: geometry collision mesh filename=./meshes/servo-hip.stl scale=0.001 0.001 0.001; visual mesh filename=./meshes/servo-hip.stl scale=0.001 0.001 0.001
- link l1_knee_servo: geometry collision mesh filename=./meshes/servo-limb-left.stl scale=0.001 0.001 0.001; visual mesh filename=./meshes/servo-limb-left.stl scale=0.001 0.001 0.001
- link l1_shoulder_servo: geometry collision mesh filename=./meshes/servo-limb-left.stl scale=0.001 0.001 0.001; visual mesh filename=./meshes/servo-limb-left.stl scale=0.001 0.001 0.001
- link l1_tibia: geometry collision mesh filename=./meshes/tibia-left.stl scale=0.001 0.001 0.001; visual mesh filename=./meshes/tibia-left.stl scale=0.001 0.001 0.001
- link l2_coxa: geometry collision mesh filename=./meshes/coxa-left.stl scale=0.001 0.001 0.001; visual mesh filename=./meshes/coxa-left.stl scale=0.001 0.001 0.001
- link l2_femur: geometry collision mesh filename=./meshes/femur-left.stl scale=0.001 0.001 0.001; visual mesh filename=./meshes/femur-left.stl scale=0.001 0.001 0.001
- link l2_hip_servo: geometry collision mesh filename=./meshes/servo-hip.stl scale=0.001 0.001 0.001; visual mesh filename=./meshes/servo-hip.stl scale=0.001 0.001 0.001
- link l2_knee_servo: geometry collision mesh filename=./meshes/servo-limb-left.stl scale=0.001 0.001 0.001; visual mesh filename=./meshes/servo-limb-left.stl scale=0.001 0.001 0.001
- link l2_shoulder_servo: geometry collision mesh filename=./meshes/servo-limb-left.stl scale=0.001 0.001 0.001; visual mesh filename=./meshes/servo-limb-left.stl scale=0.001 0.001 0.001
- link l2_tibia: geometry collision mesh filename=./meshes/tibia-left.stl scale=0.001 0.001 0.001; visual mesh filename=./meshes/tibia-left.stl scale=0.001 0.001 0.001
- link l3_coxa: geometry collision mesh filename=./meshes/coxa-left.stl scale=0.001 0.001 0.001; visual mesh filename=./meshes/coxa-left.stl scale=0.001 0.001 0.001
- link l3_femur: geometry collision mesh filename=./meshes/femur-left.stl scale=0.001 0.001 0.001; visual mesh filename=./meshes/femur-left.stl scale=0.001 0.001 0.001
- link l3_hip_servo: geometry collision mesh filename=./meshes/servo-hip.stl scale=0.001 0.001 0.001; visual mesh filename=./meshes/servo-hip.stl scale=0.001 0.001 0.001
- link l3_knee_servo: geometry collision mesh filename=./meshes/servo-limb-left.stl scale=0.001 0.001 0.001; visual mesh filename=./meshes/servo-limb-left.stl scale=0.001 0.001 0.001
- link l3_shoulder_servo: geometry collision mesh filename=./meshes/servo-limb-left.stl scale=0.001 0.001 0.001; visual mesh filename=./meshes/servo-limb-left.stl scale=0.001 0.001 0.001
- link l3_tibia: geometry collision mesh filename=./meshes/tibia-left.stl scale=0.001 0.001 0.001; visual mesh filename=./meshes/tibia-left.stl scale=0.001 0.001 0.001
- link r1_coxa: geometry collision mesh filename=./meshes/coxa-right.stl scale=0.001 0.001 0.001; visual mesh filename=./meshes/coxa-right.stl scale=0.001 0.001 0.001
- link r1_femur: geometry collision mesh filename=./meshes/femur-right.stl scale=0.001 0.001 0.001; visual mesh filename=./meshes/femur-right.stl scale=0.001 0.001 0.001
- link r1_hip_servo: geometry collision mesh filename=./meshes/servo-hip.stl scale=0.001 0.001 0.001; visual mesh filename=./meshes/servo-hip.stl scale=0.001 0.001 0.001
- link r1_knee_servo: geometry collision mesh filename=./meshes/servo-limb-right.stl scale=0.001 0.001 0.001; visual mesh filename=./meshes/servo-limb-right.stl scale=0.001 0.001 0.001
- link r1_shoulder_servo: geometry collision mesh filename=./meshes/servo-limb-right.stl scale=0.001 0.001 0.001; visual mesh filename=./meshes/servo-limb-right.stl scale=0.001 0.001 0.001
- link r1_tibia: geometry collision mesh filename=./meshes/tibia-right.stl scale=0.001 0.001 0.001; visual mesh filename=./meshes/tibia-right.stl scale=0.001 0.001 0.001
- link r2_coxa: geometry collision mesh filename=./meshes/coxa-right.stl scale=0.001 0.001 0.001; visual mesh filename=./meshes/coxa-right.stl scale=0.001 0.001 0.001
- link r2_femur: geometry collision mesh filename=./meshes/femur-right.stl scale=0.001 0.001 0.001; visual mesh filename=./meshes/femur-right.stl scale=0.001 0.001 0.001
- link r2_hip_servo: geometry collision mesh filename=./meshes/servo-hip.stl scale=0.001 0.001 0.001; visual mesh filename=./meshes/servo-hip.stl scale=0.001 0.001 0.001
- link r2_knee_servo: geometry collision mesh filename=./meshes/servo-limb-right.stl scale=0.001 0.001 0.001; visual mesh filename=./meshes/servo-limb-right.stl scale=0.001 0.001 0.001
- link r2_shoulder_servo: geometry collision mesh filename=./meshes/servo-limb-right.stl scale=0.001 0.001 0.001; visual mesh filename=./meshes/servo-limb-right.stl scale=0.001 0.001 0.001
- link r2_tibia: geometry collision mesh filename=./meshes/tibia-right.stl scale=0.001 0.001 0.001; visual mesh filename=./meshes/tibia-right.stl scale=0.001 0.001 0.001
- link r3_coxa: geometry collision mesh filename=./meshes/coxa-right.stl scale=0.001 0.001 0.001; visual mesh filename=./meshes/coxa-right.stl scale=0.001 0.001 0.001
- link r3_femur: geometry collision mesh filename=./meshes/femur-right.stl scale=0.001 0.001 0.001; visual mesh filename=./meshes/femur-right.stl scale=0.001 0.001 0.001
- link r3_hip_servo: geometry collision mesh filename=./meshes/servo-hip.stl scale=0.001 0.001 0.001; visual mesh filename=./meshes/servo-hip.stl scale=0.001 0.001 0.001
- link r3_knee_servo: geometry collision mesh filename=./meshes/servo-limb-right.stl scale=0.001 0.001 0.001; visual mesh filename=./meshes/servo-limb-right.stl scale=0.001 0.001 0.001
- link r3_shoulder_servo: geometry collision mesh filename=./meshes/servo-limb-right.stl scale=0.001 0.001 0.001; visual mesh filename=./meshes/servo-limb-right.stl scale=0.001 0.001 0.001
- link r3_tibia: geometry collision mesh filename=./meshes/tibia-right.stl scale=0.001 0.001 0.001; visual mesh filename=./meshes/tibia-right.stl scale=0.001 0.001 0.001
Joints:
- joint l1_hip: origin xyz=-0.063000 0.083500 0.000000 rpy=0.000000 0.000000 2.217165 -> xyz=-0.063000 0.083500 -0.010000 rpy=0.000000 0.000000 2.217165
- joint l1_hip_servo_joint: origin xyz=-0.063000 0.083500 0.000000 rpy=0.000000 0.000000 2.217165 -> xyz=-0.063000 0.083500 -0.010000 rpy=0.000000 0.000000 2.217165
- joint l1_tip_joint: origin xyz=0.100076 0.000000 0.000000 rpy=0.000000 0.000000 0.000000 -> xyz=0.001334 -0.004499 -0.110421 rpy=0.000000 0.000000 0.000000
- joint l2_hip: origin xyz=-0.081500 0.000000 0.000000 rpy=0.000000 0.000000 3.141593 -> xyz=-0.081500 0.000000 -0.010000 rpy=0.000000 0.000000 3.141593
- joint l2_hip_servo_joint: origin xyz=-0.081500 0.000000 0.000000 rpy=0.000000 0.000000 3.141593 -> xyz=-0.081500 0.000000 -0.010000 rpy=0.000000 0.000000 3.141593
- joint l2_tip_joint: origin xyz=0.100076 0.000000 0.000000 rpy=0.000000 0.000000 0.000000 -> xyz=0.001334 -0.004499 -0.110421 rpy=0.000000 0.000000 0.000000
- joint l3_hip: origin xyz=-0.063000 -0.083500 0.000000 rpy=0.000000 0.000000 -2.217165 -> xyz=-0.063000 -0.083500 -0.010000 rpy=0.000000 0.000000 -2.217165
- joint l3_hip_servo_joint: origin xyz=-0.063000 -0.083500 0.000000 rpy=0.000000 0.000000 -2.217165 -> xyz=-0.063000 -0.083500 -0.010000 rpy=0.000000 0.000000 -2.217165
- joint l3_tip_joint: origin xyz=0.100076 0.000000 0.000000 rpy=0.000000 0.000000 0.000000 -> xyz=0.001334 -0.004499 -0.110421 rpy=0.000000 0.000000 0.000000
- joint r1_hip: origin xyz=0.063000 0.083500 0.000000 rpy=0.000000 0.000000 0.924427 -> xyz=0.063000 0.083500 -0.010000 rpy=0.000000 0.000000 0.924427
- joint r1_hip_servo_joint: origin xyz=0.063000 0.083500 0.000000 rpy=0.000000 0.000000 0.924427 -> xyz=0.063000 0.083500 -0.010000 rpy=0.000000 0.000000 0.924427
- joint r1_tip_joint: origin xyz=0.100076 0.000000 0.000000 rpy=0.000000 0.000000 0.000000 -> xyz=0.001334 0.004499 -0.110421 rpy=0.000000 0.000000 0.000000
- joint r2_hip: origin xyz=0.081500 0.000000 0.000000 rpy=0.000000 0.000000 0.000000 -> xyz=0.081500 0.000000 -0.010000 rpy=0.000000 0.000000 0.000000
- joint r2_hip_servo_joint: origin xyz=0.081500 0.000000 0.000000 rpy=0.000000 0.000000 0.000000 -> xyz=0.081500 0.000000 -0.010000 rpy=0.000000 0.000000 0.000000
- joint r2_tip_joint: origin xyz=0.100076 0.000000 0.000000 rpy=0.000000 0.000000 0.000000 -> xyz=0.001334 0.004499 -0.110421 rpy=0.000000 0.000000 0.000000
- joint r3_hip: origin xyz=0.063000 -0.083500 0.000000 rpy=0.000000 0.000000 -0.924427 -> xyz=0.063000 -0.083500 -0.010000 rpy=0.000000 0.000000 -0.924427
- joint r3_hip_servo_joint: origin xyz=0.063000 -0.083500 0.000000 rpy=0.000000 0.000000 -0.924427 -> xyz=0.063000 -0.083500 -0.010000 rpy=0.000000 0.000000 -0.924427
- joint r3_tip_joint: origin xyz=0.100076 0.000000 0.000000 rpy=0.000000 0.000000 0.000000 -> xyz=0.001334 0.004499 -0.110421 rpy=0.000000 0.000000 0.000000

Commit message: Refactor URDF and mesh files for improved servo alignment and compatibility

File: hexapod-v2/hexapod-v2.urdf (robot description, URDF)
Before this commit: robot hexapod_v2, 43 links, 42 joints
Links:
- link base_link: geometry collision mesh filename=./meshes/bottom-cover-flat.stl scale=0.001 0.001 0.001; collision mesh filename=./meshes/frame-holes-down.stl scale=0.001 0.001 0.001
- link l1_hip_servo: geometry collision mesh filename=./meshes/servo-hip-180-lower.stl scale=0.001 0.001 0.001; visual mesh filename=./meshes/servo-hip-180-lower.stl scale=0.001 0.001 0.001
- link l2_hip_servo: geometry collision mesh filename=./meshes/servo-hip-180-lower.stl scale=0.001 0.001 0.001; visual mesh filename=./meshes/servo-hip-180-lower.stl scale=0.001 0.001 0.001
- link l3_hip_servo: geometry collision mesh filename=./meshes/servo-hip-180-lower.stl scale=0.001 0.001 0.001; visual mesh filename=./meshes/servo-hip-180-lower.stl scale=0.001 0.001 0.001
- link r1_hip_servo: geometry collision mesh filename=./meshes/servo-hip-180-lower.stl scale=0.001 0.001 0.001; visual mesh filename=./meshes/servo-hip-180-lower.stl scale=0.001 0.001 0.001
- link r2_hip_servo: geometry collision mesh filename=./meshes/servo-hip-180-lower.stl scale=0.001 0.001 0.001; visual mesh filename=./meshes/servo-hip-180-lower.stl scale=0.001 0.001 0.001
- link r3_hip_servo: geometry collision mesh filename=./meshes/servo-hip-180-lower.stl scale=0.001 0.001 0.001; visual mesh filename=./meshes/servo-hip-180-lower.stl scale=0.001 0.001 0.001

Commit message: Replace servo-hip-180-lower STL with servo-hip-shaft STL for improved alignment; update URDF references accordingly

File: hexapod-v2/hexapod-v2.urdf (robot description, URDF)
Before this commit: robot hexapod_v2, 43 links, 42 joints
Links:
- link l1_hip_servo: geometry collision mesh filename=./meshes/servo-hip-shaft.stl scale=0.001 0.001 0.001; visual mesh filename=./meshes/servo-hip-shaft.stl scale=0.001 0.001 0.001
- link l2_hip_servo: geometry collision mesh filename=./meshes/servo-hip-shaft.stl scale=0.001 0.001 0.001; visual mesh filename=./meshes/servo-hip-shaft.stl scale=0.001 0.001 0.001
- link l3_hip_servo: geometry collision mesh filename=./meshes/servo-hip-shaft.stl scale=0.001 0.001 0.001; visual mesh filename=./meshes/servo-hip-shaft.stl scale=0.001 0.001 0.001
- link r1_hip_servo: geometry collision mesh filename=./meshes/servo-hip-shaft.stl scale=0.001 0.001 0.001; visual mesh filename=./meshes/servo-hip-shaft.stl scale=0.001 0.001 0.001
- link r2_hip_servo: geometry collision mesh filename=./meshes/servo-hip-shaft.stl scale=0.001 0.001 0.001; visual mesh filename=./meshes/servo-hip-shaft.stl scale=0.001 0.001 0.001
- link r3_hip_servo: geometry collision mesh filename=./meshes/servo-hip-shaft.stl scale=0.001 0.001 0.001; visual mesh filename=./meshes/servo-hip-shaft.stl scale=0.001 0.001 0.001

Commit message: Refactor leg frame definitions and update hip joint origins for improved alignment in URDF

File: hexapod-v2/hexapod-v2.urdf (robot description, URDF)
Before this commit: robot hexapod_v2, 43 links, 42 joints
Joints:
- joint l1_hip: origin xyz=-0.063000 0.083500 -0.010000 rpy=0.000000 0.000000 2.217165 -> xyz=-0.076600 0.084571 -0.010000 rpy=0.000000 0.000000 2.356194
- joint l1_hip_servo_joint: origin xyz=-0.063000 0.083500 -0.010000 rpy=0.000000 0.000000 2.217165 -> xyz=-0.076600 0.084571 -0.010000 rpy=0.000000 0.000000 2.356194
- joint l2_hip: origin xyz=-0.081500 0.000000 -0.010000 rpy=0.000000 0.000000 3.141593 -> xyz=-0.091000 -0.008029 -0.010000 rpy=0.000000 0.000000 3.141593
- joint l2_hip_servo_joint: origin xyz=-0.081500 0.000000 -0.010000 rpy=0.000000 0.000000 3.141593 -> xyz=-0.091000 -0.008029 -0.010000 rpy=0.000000 0.000000 3.141593
- joint l3_hip: origin xyz=-0.063000 -0.083500 -0.010000 rpy=0.000000 0.000000 -2.217165 -> xyz=-0.062547 -0.094718 -0.010000 rpy=0.000000 0.000000 -2.356176
- joint l3_hip_servo_joint: origin xyz=-0.063000 -0.083500 -0.010000 rpy=0.000000 0.000000 -2.217165 -> xyz=-0.062547 -0.094718 -0.010000 rpy=0.000000 0.000000 -2.356176
- joint r1_hip: origin xyz=0.063000 0.083500 -0.010000 rpy=0.000000 0.000000 0.924427 -> xyz=0.076600 0.084571 -0.010000 rpy=0.000000 0.000000 0.785398
- joint r1_hip_servo_joint: origin xyz=0.063000 0.083500 -0.010000 rpy=0.000000 0.000000 0.924427 -> xyz=0.076600 0.084571 -0.010000 rpy=0.000000 0.000000 0.785398
- joint r2_hip: origin xyz=0.081500 0.000000 -0.010000 rpy=0.000000 0.000000 0.000000 -> xyz=0.091000 -0.008029 -0.010000 rpy=0.000000 0.000000 0.000000
- joint r2_hip_servo_joint: origin xyz=0.081500 0.000000 -0.010000 rpy=0.000000 0.000000 0.000000 -> xyz=0.091000 -0.008029 -0.010000 rpy=0.000000 0.000000 0.000000
- joint r3_hip: origin xyz=0.063000 -0.083500 -0.010000 rpy=0.000000 0.000000 -0.924427 -> xyz=0.062547 -0.094718 -0.010000 rpy=0.000000 0.000000 -0.785416
- joint r3_hip_servo_joint: origin xyz=0.063000 -0.083500 -0.010000 rpy=0.000000 0.000000 -0.924427 -> xyz=0.062547 -0.094718 -0.010000 rpy=0.000000 0.000000 -0.785416

Commit message: Refactor servo mounting logic and update URDF joint origins for improved alignment

File: hexapod-v2/hexapod-v2.urdf (robot description, URDF)
Before this commit: robot hexapod_v2, 43 links, 42 joints
Joints:
- joint l1_hip: origin xyz=-0.076600 0.084571 -0.010000 rpy=0.000000 0.000000 2.356194 -> xyz=-0.062862 0.084988 -0.010000 rpy=0.000000 0.000000 2.356194
- joint l1_hip_servo_joint: origin xyz=-0.076600 0.084571 -0.010000 rpy=0.000000 0.000000 2.356194 -> xyz=-0.062862 0.084988 -0.010000 rpy=0.000000 0.000000 2.356194
- joint l2_hip: origin xyz=-0.091000 -0.008029 -0.010000 rpy=0.000000 0.000000 3.141593 -> xyz=-0.081580 0.001980 -0.010000 rpy=0.000000 0.000000 3.141593
- joint l2_hip_servo_joint: origin xyz=-0.091000 -0.008029 -0.010000 rpy=0.000000 0.000000 3.141593 -> xyz=-0.081580 0.001980 -0.010000 rpy=0.000000 0.000000 3.141593
- joint l3_hip: origin xyz=-0.062547 -0.094718 -0.010000 rpy=0.000000 0.000000 -2.356176 -> xyz=-0.062851 -0.081010 -0.010000 rpy=0.000000 0.000000 -2.356176
- joint l3_hip_servo_joint: origin xyz=-0.062547 -0.094718 -0.010000 rpy=0.000000 0.000000 -2.356176 -> xyz=-0.062851 -0.081010 -0.010000 rpy=0.000000 0.000000 -2.356176
- joint r1_hip: origin xyz=0.076600 0.084571 -0.010000 rpy=0.000000 0.000000 0.785398 -> xyz=0.062874 0.084976 -0.010000 rpy=0.000000 0.000000 0.785398
- joint r1_hip_servo_joint: origin xyz=0.076600 0.084571 -0.010000 rpy=0.000000 0.000000 0.785398 -> xyz=0.062874 0.084976 -0.010000 rpy=0.000000 0.000000 0.785398
- joint r2_hip: origin xyz=0.091000 -0.008029 -0.010000 rpy=0.000000 0.000000 0.000000 -> xyz=0.081580 0.001962 -0.010000 rpy=0.000000 0.000000 0.000000
- joint r2_hip_servo_joint: origin xyz=0.091000 -0.008029 -0.010000 rpy=0.000000 0.000000 0.000000 -> xyz=0.081580 0.001962 -0.010000 rpy=0.000000 0.000000 0.000000
- joint r3_hip: origin xyz=0.062547 -0.094718 -0.010000 rpy=0.000000 0.000000 -0.785416 -> xyz=0.062839 -0.081022 -0.010000 rpy=0.000000 0.000000 -0.785416
- joint r3_hip_servo_joint: origin xyz=0.062547 -0.094718 -0.010000 rpy=0.000000 0.000000 -0.785416 -> xyz=0.062839 -0.081022 -0.010000 rpy=0.000000 0.000000 -0.785416

Commit message: Add tibia proximal axis definition and update URDF joint references for improved alignment

File: hexapod-v2/hexapod-v2.urdf (robot description, URDF)
Before this commit: robot hexapod_v2, 43 links, 42 joints
Joints:
- joint l1_knee: origin xyz=0.080000 0.000000 0.000000 rpy=0.000000 0.000000 0.000000 -> xyz=0.000000 0.000000 0.000000 rpy=0.000000 0.000000 0.000000; parent l1_femur -> l1_knee_servo
- joint l1_tip_joint: origin xyz=0.001334 -0.004499 -0.110421 rpy=0.000000 0.000000 0.000000 -> xyz=-0.050423 -0.004499 -0.119208 rpy=0.000000 0.000000 0.000000
- joint l2_knee: origin xyz=0.080000 0.000000 0.000000 rpy=0.000000 0.000000 0.000000 -> xyz=0.000000 0.000000 0.000000 rpy=0.000000 0.000000 0.000000; parent l2_femur -> l2_knee_servo
- joint l2_tip_joint: origin xyz=0.001334 -0.004499 -0.110421 rpy=0.000000 0.000000 0.000000 -> xyz=-0.050423 -0.004499 -0.119208 rpy=0.000000 0.000000 0.000000
- joint l3_knee: origin xyz=0.080000 0.000000 0.000000 rpy=0.000000 0.000000 0.000000 -> xyz=0.000000 0.000000 0.000000 rpy=0.000000 0.000000 0.000000; parent l3_femur -> l3_knee_servo
- joint l3_tip_joint: origin xyz=0.001334 -0.004499 -0.110421 rpy=0.000000 0.000000 0.000000 -> xyz=-0.050423 -0.004499 -0.119208 rpy=0.000000 0.000000 0.000000
- joint r1_knee: origin xyz=0.080000 0.000000 0.000000 rpy=0.000000 0.000000 0.000000 -> xyz=0.000000 0.000000 0.000000 rpy=0.000000 0.000000 0.000000; parent r1_femur -> r1_knee_servo
- joint r1_tip_joint: origin xyz=0.001334 0.004499 -0.110421 rpy=0.000000 0.000000 0.000000 -> xyz=-0.050423 0.004499 -0.119208 rpy=0.000000 0.000000 0.000000
- joint r2_knee: origin xyz=0.080000 0.000000 0.000000 rpy=0.000000 0.000000 0.000000 -> xyz=0.000000 0.000000 0.000000 rpy=0.000000 0.000000 0.000000; parent r2_femur -> r2_knee_servo
- joint r2_tip_joint: origin xyz=0.001334 0.004499 -0.110421 rpy=0.000000 0.000000 0.000000 -> xyz=-0.050423 0.004499 -0.119208 rpy=0.000000 0.000000 0.000000
- joint r3_knee: origin xyz=0.080000 0.000000 0.000000 rpy=0.000000 0.000000 0.000000 -> xyz=0.000000 0.000000 0.000000 rpy=0.000000 0.000000 0.000000; parent r3_femur -> r3_knee_servo
- joint r3_tip_joint: origin xyz=0.001334 0.004499 -0.110421 rpy=0.000000 0.000000 0.000000 -> xyz=-0.050423 0.004499 -0.119208 rpy=0.000000 0.000000 0.000000

Commit message: Update knee joint definitions in URDF for improved articulation and dynamics

File: hexapod-v2/hexapod-v2.urdf (robot description, URDF)
Before this commit: robot hexapod_v2, 43 links, 42 joints
Joints:
- removed joint l1_knee_servo_joint
- removed joint l2_knee_servo_joint
- removed joint l3_knee_servo_joint
- removed joint r1_knee_servo_joint
- removed joint r2_knee_servo_joint
- removed joint r3_knee_servo_joint
- added joint l1_tibia_mount_joint: type fixed, parent l1_knee_servo, child l1_tibia, origin xyz=0.000000 0.000000 0.000000 rpy=0.000000 0.000000 0.000000
- added joint l2_tibia_mount_joint: type fixed, parent l2_knee_servo, child l2_tibia, origin xyz=0.000000 0.000000 0.000000 rpy=0.000000 0.000000 0.000000
- added joint l3_tibia_mount_joint: type fixed, parent l3_knee_servo, child l3_tibia, origin xyz=0.000000 0.000000 0.000000 rpy=0.000000 0.000000 0.000000
- added joint r1_tibia_mount_joint: type fixed, parent r1_knee_servo, child r1_tibia, origin xyz=0.000000 0.000000 0.000000 rpy=0.000000 0.000000 0.000000
- added joint r2_tibia_mount_joint: type fixed, parent r2_knee_servo, child r2_tibia, origin xyz=0.000000 0.000000 0.000000 rpy=0.000000 0.000000 0.000000
- added joint r3_tibia_mount_joint: type fixed, parent r3_knee_servo, child r3_tibia, origin xyz=0.000000 0.000000 0.000000 rpy=0.000000 0.000000 0.000000
- joint l1_knee: child l1_tibia -> l1_knee_servo; origin xyz=0.000000 0.000000 0.000000 rpy=0.000000 0.000000 0.000000 -> xyz=0.080000 0.000000 0.000000 rpy=0.000000 0.000000 0.000000; parent l1_knee_servo -> l1_femur
- joint l2_knee: child l2_tibia -> l2_knee_servo; origin xyz=0.000000 0.000000 0.000000 rpy=0.000000 0.000000 0.000000 -> xyz=0.080000 0.000000 0.000000 rpy=0.000000 0.000000 0.000000; parent l2_knee_servo -> l2_femur
- joint l3_knee: child l3_tibia -> l3_knee_servo; origin xyz=0.000000 0.000000 0.000000 rpy=0.000000 0.000000 0.000000 -> xyz=0.080000 0.000000 0.000000 rpy=0.000000 0.000000 0.000000; parent l3_knee_servo -> l3_femur
- joint r1_knee: child r1_tibia -> r1_knee_servo; origin xyz=0.000000 0.000000 0.000000 rpy=0.000000 0.000000 0.000000 -> xyz=0.080000 0.000000 0.000000 rpy=0.000000 0.000000 0.000000; parent r1_knee_servo -> r1_femur
- joint r2_knee: child r2_tibia -> r2_knee_servo; origin xyz=0.000000 0.000000 0.000000 rpy=0.000000 0.000000 0.000000 -> xyz=0.080000 0.000000 0.000000 rpy=0.000000 0.000000 0.000000; parent r2_knee_servo -> r2_femur
- joint r3_knee: child r3_tibia -> r3_knee_servo; origin xyz=0.000000 0.000000 0.000000 rpy=0.000000 0.000000 0.000000 -> xyz=0.080000 0.000000 0.000000 rpy=0.000000 0.000000 0.000000; parent r3_knee_servo -> r3_femur

Commit message: Add rotation function for Y-axis and update tibia mesh orientations in URDF for improved alignment

File: hexapod-v2/hexapod-v2.urdf (robot description, URDF)
Before this commit: robot hexapod_v2, 43 links, 42 joints
Joints:
- joint l1_tip_joint: origin xyz=-0.050423 -0.004499 -0.119208 rpy=0.000000 0.000000 0.000000 -> xyz=0.050423 0.004499 -0.119208 rpy=0.000000 0.000000 0.000000
- joint l2_tip_joint: origin xyz=-0.050423 -0.004499 -0.119208 rpy=0.000000 0.000000 0.000000 -> xyz=0.050423 0.004499 -0.119208 rpy=0.000000 0.000000 0.000000
- joint l3_tip_joint: origin xyz=-0.050423 -0.004499 -0.119208 rpy=0.000000 0.000000 0.000000 -> xyz=0.050423 0.004499 -0.119208 rpy=0.000000 0.000000 0.000000
- joint r1_tip_joint: origin xyz=-0.050423 0.004499 -0.119208 rpy=0.000000 0.000000 0.000000 -> xyz=0.050423 -0.004499 -0.119208 rpy=0.000000 0.000000 0.000000
- joint r2_tip_joint: origin xyz=-0.050423 0.004499 -0.119208 rpy=0.000000 0.000000 0.000000 -> xyz=0.050423 -0.004499 -0.119208 rpy=0.000000 0.000000 0.000000
- joint r3_tip_joint: origin xyz=-0.050423 0.004499 -0.119208 rpy=0.000000 0.000000 0.000000 -> xyz=0.050423 -0.004499 -0.119208 rpy=0.000000 0.000000 0.000000
