Commit message: Adjust BODY_Z parameter and update hip servo orientations in URDF for improved alignment

File: hexapod-v2/hexapod-v2.urdf (robot description, URDF)
Before this commit: robot hexapod_v2, 43 links, 42 joints
Joints:
- joint l1_hip: origin xyz=-0.062862 0.084988 -0.010000 rpy=0.000000 0.000000 2.356194 -> xyz=-0.062862 0.084988 -0.008000 rpy=0.000000 0.000000 2.356194
- joint l1_hip_servo_joint: origin xyz=-0.062862 0.084988 -0.010000 rpy=0.000000 0.000000 2.356194 -> xyz=-0.062862 0.084988 -0.008000 rpy=0.000000 0.000000 2.356194
- joint l2_hip: origin xyz=-0.081580 0.001980 -0.010000 rpy=0.000000 0.000000 3.141593 -> xyz=-0.081580 0.001980 -0.008000 rpy=0.000000 0.000000 3.141593
- joint l2_hip_servo_joint: origin xyz=-0.081580 0.001980 -0.010000 rpy=0.000000 0.000000 3.141593 -> xyz=-0.081580 0.001980 -0.008000 rpy=0.000000 0.000000 3.141593
- joint l3_hip: origin xyz=-0.062851 -0.081010 -0.010000 rpy=0.000000 0.000000 -2.356176 -> xyz=-0.062851 -0.081010 -0.008000 rpy=0.000000 0.000000 -2.356176
- joint l3_hip_servo_joint: origin xyz=-0.062851 -0.081010 -0.010000 rpy=0.000000 0.000000 -2.356176 -> xyz=-0.062851 -0.081010 -0.008000 rpy=0.000000 0.000000 -2.356176
- joint r1_hip: origin xyz=0.062874 0.084976 -0.010000 rpy=0.000000 0.000000 0.785398 -> xyz=0.062874 0.084976 -0.008000 rpy=0.000000 0.000000 0.785398
- joint r1_hip_servo_joint: origin xyz=0.062874 0.084976 -0.010000 rpy=0.000000 0.000000 0.785398 -> xyz=0.062874 0.084976 -0.008000 rpy=0.000000 0.000000 0.785398
- joint r2_hip: origin xyz=0.081580 0.001962 -0.010000 rpy=0.000000 0.000000 0.000000 -> xyz=0.081580 0.001962 -0.008000 rpy=0.000000 0.000000 0.000000
- joint r2_hip_servo_joint: origin xyz=0.081580 0.001962 -0.010000 rpy=0.000000 0.000000 0.000000 -> xyz=0.081580 0.001962 -0.008000 rpy=0.000000 0.000000 0.000000
- joint r3_hip: origin xyz=0.062839 -0.081022 -0.010000 rpy=0.000000 0.000000 -0.785416 -> xyz=0.062839 -0.081022 -0.008000 rpy=0.000000 0.000000 -0.785416
- joint r3_hip_servo_joint: origin xyz=0.062839 -0.081022 -0.010000 rpy=0.000000 0.000000 -0.785416 -> xyz=0.062839 -0.081022 -0.008000 rpy=0.000000 0.000000 -0.785416

Commit message: Refactor servo mount calculations and update shoulder joint origins for improved accuracy in URDF

File: hexapod-v2/hexapod-v2.urdf (robot description, URDF)
Before this commit: robot hexapod_v2, 43 links, 42 joints
Joints:
- joint l1_shoulder: origin xyz=0.043000 0.000000 0.000000 rpy=0.000000 0.000000 0.000000 -> xyz=0.042992 0.000000 0.000420 rpy=0.000000 0.000000 0.000000
- joint l1_shoulder_servo_joint: origin xyz=0.043000 0.000000 0.000000 rpy=0.000000 0.000000 0.000000 -> xyz=0.042992 0.000000 0.000420 rpy=0.000000 0.000000 0.000000
- joint l2_shoulder: origin xyz=0.043000 0.000000 0.000000 rpy=0.000000 0.000000 0.000000 -> xyz=0.042992 0.000000 0.000420 rpy=0.000000 0.000000 0.000000
- joint l2_shoulder_servo_joint: origin xyz=0.043000 0.000000 0.000000 rpy=0.000000 0.000000 0.000000 -> xyz=0.042992 0.000000 0.000420 rpy=0.000000 0.000000 0.000000
- joint l3_shoulder: origin xyz=0.043000 0.000000 0.000000 rpy=0.000000 0.000000 0.000000 -> xyz=0.042992 0.000000 0.000420 rpy=0.000000 0.000000 0.000000
- joint l3_shoulder_servo_joint: origin xyz=0.043000 0.000000 0.000000 rpy=0.000000 0.000000 0.000000 -> xyz=0.042992 0.000000 0.000420 rpy=0.000000 0.000000 0.000000
- joint r1_shoulder: origin xyz=0.043000 0.000000 0.000000 rpy=0.000000 0.000000 0.000000 -> xyz=0.043008 0.000000 0.000420 rpy=0.000000 0.000000 0.000000
- joint r1_shoulder_servo_joint: origin xyz=0.043000 0.000000 0.000000 rpy=0.000000 0.000000 0.000000 -> xyz=0.043008 0.000000 0.000420 rpy=0.000000 0.000000 0.000000
- joint r2_shoulder: origin xyz=0.043000 0.000000 0.000000 rpy=0.000000 0.000000 0.000000 -> xyz=0.043008 0.000000 0.000420 rpy=0.000000 0.000000 0.000000
- joint r2_shoulder_servo_joint: origin xyz=0.043000 0.000000 0.000000 rpy=0.000000 0.000000 0.000000 -> xyz=0.043008 0.000000 0.000420 rpy=0.000000 0.000000 0.000000
- joint r3_shoulder: origin xyz=0.043000 0.000000 0.000000 rpy=0.000000 0.000000 0.000000 -> xyz=0.043008 0.000000 0.000420 rpy=0.000000 0.000000 0.000000
- joint r3_shoulder_servo_joint: origin xyz=0.043000 0.000000 0.000000 rpy=0.000000 0.000000 0.000000 -> xyz=0.043008 0.000000 0.000420 rpy=0.000000 0.000000 0.000000

Commit message: Add tibia knee mount hole coordinates and rotation functions; update URDF joint origins for improved alignment

File: hexapod-v2/hexapod-v2.urdf (robot description, URDF)
Before this commit: robot hexapod_v2, 43 links, 42 joints
Joints:
- joint l1_tip_joint: origin xyz=0.050423 0.004499 -0.119208 rpy=0.000000 0.000000 0.000000 -> xyz=0.022531 0.004531 -0.095727 rpy=0.000000 0.000000 0.000000
- joint l2_tip_joint: origin xyz=0.050423 0.004499 -0.119208 rpy=0.000000 0.000000 0.000000 -> xyz=0.022531 0.004531 -0.095727 rpy=0.000000 0.000000 0.000000
- joint l3_tip_joint: origin xyz=0.050423 0.004499 -0.119208 rpy=0.000000 0.000000 0.000000 -> xyz=0.022531 0.004531 -0.095727 rpy=0.000000 0.000000 0.000000
- joint r1_tip_joint: origin xyz=0.050423 -0.004499 -0.119208 rpy=0.000000 0.000000 0.000000 -> xyz=0.022514 -0.004531 -0.095727 rpy=0.000000 0.000000 0.000000
- joint r2_tip_joint: origin xyz=0.050423 -0.004499 -0.119208 rpy=0.000000 0.000000 0.000000 -> xyz=0.022514 -0.004531 -0.095727 rpy=0.000000 0.000000 0.000000
- joint r3_tip_joint: origin xyz=0.050423 -0.004499 -0.119208 rpy=0.000000 0.000000 0.000000 -> xyz=0.022514 -0.004531 -0.095727 rpy=0.000000 0.000000 0.000000

Commit message: Update femur dimensions and adjust URDF joint origins for improved alignment; replace femur mesh files

File: hexapod-v2/hexapod-v2.urdf (robot description, URDF)
Before this commit: robot hexapod_v2, 43 links, 42 joints
Joints:
- joint l1_knee: origin xyz=0.080000 0.000000 0.000000 rpy=0.000000 0.000000 0.000000 -> xyz=0.060000 0.000000 0.000000 rpy=0.000000 0.000000 0.000000
- joint l2_knee: origin xyz=0.080000 0.000000 0.000000 rpy=0.000000 0.000000 0.000000 -> xyz=0.060000 0.000000 0.000000 rpy=0.000000 0.000000 0.000000
- joint l3_knee: origin xyz=0.080000 0.000000 0.000000 rpy=0.000000 0.000000 0.000000 -> xyz=0.060000 0.000000 0.000000 rpy=0.000000 0.000000 0.000000
- joint r1_knee: origin xyz=0.080000 0.000000 0.000000 rpy=0.000000 0.000000 0.000000 -> xyz=0.060000 0.000000 0.000000 rpy=0.000000 0.000000 0.000000
- joint r2_knee: origin xyz=0.080000 0.000000 0.000000 rpy=0.000000 0.000000 0.000000 -> xyz=0.060000 0.000000 0.000000 rpy=0.000000 0.000000 0.000000
- joint r3_knee: origin xyz=0.080000 0.000000 0.000000 rpy=0.000000 0.000000 0.000000 -> xyz=0.060000 0.000000 0.000000 rpy=0.000000 0.000000 0.000000

Commit message: Add knee and shoulder servo configurations and update URDF
- Introduced KNEE_SERVO_ROTATIONS and SHOULDER_SERVO_ROTATIONS for proper alignment of knee and shoulder servos.
- Updated shoulder and knee servo references in the URDF generation logic.
- Added new STL files for knee and shoulder servos with 180-degree rotation.
- Adjusted joint definitions in the URDF to reflect the new servo configurations and corrected origin positions.
- Updated existing STL references in the URDF to point to the new servo models.

File: hexapod-v2/hexapod-v2.urdf (robot description, URDF)
Before this commit: robot hexapod_v2, 43 links, 42 joints
Links:
- link l1_knee_servo: geometry collision mesh filename=./meshes/servo-knee-left.stl scale=0.001 0.001 0.001; visual mesh filename=./meshes/servo-knee-left.stl scale=0.001 0.001 0.001
- link l1_shoulder_servo: geometry collision mesh filename=./meshes/servo-shoulder-rot180-left.stl scale=0.001 0.001 0.001; visual mesh filename=./meshes/servo-shoulder-rot180-left.stl scale=0.001 0.001 0.001
- link l2_knee_servo: geometry collision mesh filename=./meshes/servo-knee-left.stl scale=0.001 0.001 0.001; visual mesh filename=./meshes/servo-knee-left.stl scale=0.001 0.001 0.001
- link l2_shoulder_servo: geometry collision mesh filename=./meshes/servo-shoulder-rot180-left.stl scale=0.001 0.001 0.001; visual mesh filename=./meshes/servo-shoulder-rot180-left.stl scale=0.001 0.001 0.001
- link l3_knee_servo: geometry collision mesh filename=./meshes/servo-knee-left.stl scale=0.001 0.001 0.001; visual mesh filename=./meshes/servo-knee-left.stl scale=0.001 0.001 0.001
- link l3_shoulder_servo: geometry collision mesh filename=./meshes/servo-shoulder-rot180-left.stl scale=0.001 0.001 0.001; visual mesh filename=./meshes/servo-shoulder-rot180-left.stl scale=0.001 0.001 0.001
- link r1_knee_servo: geometry collision mesh filename=./meshes/servo-knee-right.stl scale=0.001 0.001 0.001; visual mesh filename=./meshes/servo-knee-right.stl scale=0.001 0.001 0.001
- link r1_shoulder_servo: geometry collision mesh filename=./meshes/servo-shoulder-rot180-right.stl scale=0.001 0.001 0.001; visual mesh filename=./meshes/servo-shoulder-rot180-right.stl scale=0.001 0.001 0.001
- link r2_knee_servo: geometry collision mesh filename=./meshes/servo-knee-right.stl scale=0.001 0.001 0.001; visual mesh filename=./meshes/servo-knee-right.stl scale=0.001 0.001 0.001
- link r2_shoulder_servo: geometry collision mesh filename=./meshes/servo-shoulder-rot180-right.stl scale=0.001 0.001 0.001; visual mesh filename=./meshes/servo-shoulder-rot180-right.stl scale=0.001 0.001 0.001
- link r3_knee_servo: geometry collision mesh filename=./meshes/servo-knee-right.stl scale=0.001 0.001 0.001; visual mesh filename=./meshes/servo-knee-right.stl scale=0.001 0.001 0.001
- link r3_shoulder_servo: geometry collision mesh filename=./meshes/servo-shoulder-rot180-right.stl scale=0.001 0.001 0.001; visual mesh filename=./meshes/servo-shoulder-rot180-right.stl scale=0.001 0.001 0.001
Joints:
- removed joint l1_tibia_mount_joint
- removed joint l2_tibia_mount_joint
- removed joint l3_tibia_mount_joint
- removed joint r1_tibia_mount_joint
- removed joint r2_tibia_mount_joint
- removed joint r3_tibia_mount_joint
- added joint l1_knee_servo_joint: type fixed, parent l1_femur, child l1_knee_servo, origin xyz=0.060000 0.000000 0.000000 rpy=0.000000 0.000000 0.000000
- added joint l2_knee_servo_joint: type fixed, parent l2_femur, child l2_knee_servo, origin xyz=0.060000 0.000000 0.000000 rpy=0.000000 0.000000 0.000000
- added joint l3_knee_servo_joint: type fixed, parent l3_femur, child l3_knee_servo, origin xyz=0.060000 0.000000 0.000000 rpy=0.000000 0.000000 0.000000
- added joint r1_knee_servo_joint: type fixed, parent r1_femur, child r1_knee_servo, origin xyz=0.060000 0.000000 0.000000 rpy=0.000000 0.000000 0.000000
- added joint r2_knee_servo_joint: type fixed, parent r2_femur, child r2_knee_servo, origin xyz=0.060000 0.000000 0.000000 rpy=0.000000 0.000000 0.000000
- added joint r3_knee_servo_joint: type fixed, parent r3_femur, child r3_knee_servo, origin xyz=0.060000 0.000000 0.000000 rpy=0.000000 0.000000 0.000000
- joint l1_knee: child l1_knee_servo -> l1_tibia
- joint l1_shoulder: origin xyz=0.042992 0.000000 0.000420 rpy=0.000000 0.000000 0.000000 -> xyz=0.042992 0.000000 0.020580 rpy=0.000000 0.000000 0.000000
- joint l1_shoulder_servo_joint: origin xyz=0.042992 0.000000 0.000420 rpy=0.000000 0.000000 0.000000 -> xyz=0.042992 0.000000 0.020580 rpy=0.000000 0.000000 0.000000
- joint l1_tip_joint: origin xyz=0.022531 0.004531 -0.095727 rpy=0.000000 0.000000 0.000000 -> xyz=0.022514 0.004531 -0.095727 rpy=0.000000 0.000000 0.000000
- joint l2_knee: child l2_knee_servo -> l2_tibia
- joint l2_shoulder: origin xyz=0.042992 0.000000 0.000420 rpy=0.000000 0.000000 0.000000 -> xyz=0.042992 0.000000 0.020580 rpy=0.000000 0.000000 0.000000
- joint l2_shoulder_servo_joint: origin xyz=0.042992 0.000000 0.000420 rpy=0.000000 0.000000 0.000000 -> xyz=0.042992 0.000000 0.020580 rpy=0.000000 0.000000 0.000000
- joint l2_tip_joint: origin xyz=0.022531 0.004531 -0.095727 rpy=0.000000 0.000000 0.000000 -> xyz=0.022514 0.004531 -0.095727 rpy=0.000000 0.000000 0.000000
- joint l3_knee: child l3_knee_servo -> l3_tibia
- joint l3_shoulder: origin xyz=0.042992 0.000000 0.000420 rpy=0.000000 0.000000 0.000000 -> xyz=0.042992 0.000000 0.020580 rpy=0.000000 0.000000 0.000000
- joint l3_shoulder_servo_joint: origin xyz=0.042992 0.000000 0.000420 rpy=0.000000 0.000000 0.000000 -> xyz=0.042992 0.000000 0.020580 rpy=0.000000 0.000000 0.000000
- joint l3_tip_joint: origin xyz=0.022531 0.004531 -0.095727 rpy=0.000000 0.000000 0.000000 -> xyz=0.022514 0.004531 -0.095727 rpy=0.000000 0.000000 0.000000
- joint r1_knee: child r1_knee_servo -> r1_tibia
- joint r1_shoulder: origin xyz=0.043008 0.000000 0.000420 rpy=0.000000 0.000000 0.000000 -> xyz=0.043008 0.000000 0.020580 rpy=0.000000 0.000000 0.000000
- joint r1_shoulder_servo_joint: origin xyz=0.043008 0.000000 0.000420 rpy=0.000000 0.000000 0.000000 -> xyz=0.043008 0.000000 0.020580 rpy=0.000000 0.000000 0.000000
- joint r1_tip_joint: origin xyz=0.022514 -0.004531 -0.095727 rpy=0.000000 0.000000 0.000000 -> xyz=0.022531 -0.004531 -0.095727 rpy=0.000000 0.000000 0.000000
- joint r2_knee: child r2_knee_servo -> r2_tibia
- joint r2_shoulder: origin xyz=0.043008 0.000000 0.000420 rpy=0.000000 0.000000 0.000000 -> xyz=0.043008 0.000000 0.020580 rpy=0.000000 0.000000 0.000000
- joint r2_shoulder_servo_joint: origin xyz=0.043008 0.000000 0.000420 rpy=0.000000 0.000000 0.000000 -> xyz=0.043008 0.000000 0.020580 rpy=0.000000 0.000000 0.000000
- joint r2_tip_joint: origin xyz=0.022514 -0.004531 -0.095727 rpy=0.000000 0.000000 0.000000 -> xyz=0.022531 -0.004531 -0.095727 rpy=0.000000 0.000000 0.000000
- joint r3_knee: child r3_knee_servo -> r3_tibia
- joint r3_shoulder: origin xyz=0.043008 0.000000 0.000420 rpy=0.000000 0.000000 0.000000 -> xyz=0.043008 0.000000 0.020580 rpy=0.000000 0.000000 0.000000
- joint r3_shoulder_servo_joint: origin xyz=0.043008 0.000000 0.000420 rpy=0.000000 0.000000 0.000000 -> xyz=0.043008 0.000000 0.020580 rpy=0.000000 0.000000 0.000000
- joint r3_tip_joint: origin xyz=0.022514 -0.004531 -0.095727 rpy=0.000000 0.000000 0.000000 -> xyz=0.022531 -0.004531 -0.095727 rpy=0.000000 0.000000 0.000000

Commit message: Update shoulder servo mesh files and adjust URDF for correct rotation; replace old mesh references

File: hexapod-v2/hexapod-v2.urdf (robot description, URDF)
Before this commit: robot hexapod_v2, 43 links, 42 joints
Links:
- link l1_shoulder_servo: geometry collision mesh filename=./meshes/servo-shoulder-z180-left.stl scale=0.001 0.001 0.001; visual mesh filename=./meshes/servo-shoulder-z180-left.stl scale=0.001 0.001 0.001
- link l2_shoulder_servo: geometry collision mesh filename=./meshes/servo-shoulder-z180-left.stl scale=0.001 0.001 0.001; visual mesh filename=./meshes/servo-shoulder-z180-left.stl scale=0.001 0.001 0.001
- link l3_shoulder_servo: geometry collision mesh filename=./meshes/servo-shoulder-z180-left.stl scale=0.001 0.001 0.001; visual mesh filename=./meshes/servo-shoulder-z180-left.stl scale=0.001 0.001 0.001
- link r1_shoulder_servo: geometry collision mesh filename=./meshes/servo-shoulder-z180-right.stl scale=0.001 0.001 0.001; visual mesh filename=./meshes/servo-shoulder-z180-right.stl scale=0.001 0.001 0.001
- link r2_shoulder_servo: geometry collision mesh filename=./meshes/servo-shoulder-z180-right.stl scale=0.001 0.001 0.001; visual mesh filename=./meshes/servo-shoulder-z180-right.stl scale=0.001 0.001 0.001
- link r3_shoulder_servo: geometry collision mesh filename=./meshes/servo-shoulder-z180-right.stl scale=0.001 0.001 0.001; visual mesh filename=./meshes/servo-shoulder-z180-right.stl scale=0.001 0.001 0.001
Joints:
- joint l1_shoulder: origin xyz=0.042992 0.000000 0.020580 rpy=0.000000 0.000000 0.000000 -> xyz=0.043008 0.000000 0.000420 rpy=0.000000 0.000000 0.000000
- joint l1_shoulder_servo_joint: origin xyz=0.042992 0.000000 0.020580 rpy=0.000000 0.000000 0.000000 -> xyz=0.043008 0.000000 0.000420 rpy=0.000000 0.000000 0.000000
- joint l2_shoulder: origin xyz=0.042992 0.000000 0.020580 rpy=0.000000 0.000000 0.000000 -> xyz=0.043008 0.000000 0.000420 rpy=0.000000 0.000000 0.000000
- joint l2_shoulder_servo_joint: origin xyz=0.042992 0.000000 0.020580 rpy=0.000000 0.000000 0.000000 -> xyz=0.043008 0.000000 0.000420 rpy=0.000000 0.000000 0.000000
- joint l3_shoulder: origin xyz=0.042992 0.000000 0.020580 rpy=0.000000 0.000000 0.000000 -> xyz=0.043008 0.000000 0.000420 rpy=0.000000 0.000000 0.000000
- joint l3_shoulder_servo_joint: origin xyz=0.042992 0.000000 0.020580 rpy=0.000000 0.000000 0.000000 -> xyz=0.043008 0.000000 0.000420 rpy=0.000000 0.000000 0.000000
- joint r1_shoulder: origin xyz=0.043008 0.000000 0.020580 rpy=0.000000 0.000000 0.000000 -> xyz=0.042992 0.000000 0.000420 rpy=0.000000 0.000000 0.000000
- joint r1_shoulder_servo_joint: origin xyz=0.043008 0.000000 0.020580 rpy=0.000000 0.000000 0.000000 -> xyz=0.042992 0.000000 0.000420 rpy=0.000000 0.000000 0.000000
- joint r2_shoulder: origin xyz=0.043008 0.000000 0.020580 rpy=0.000000 0.000000 0.000000 -> xyz=0.042992 0.000000 0.000420 rpy=0.000000 0.000000 0.000000
- joint r2_shoulder_servo_joint: origin xyz=0.043008 0.000000 0.020580 rpy=0.000000 0.000000 0.000000 -> xyz=0.042992 0.000000 0.000420 rpy=0.000000 0.000000 0.000000
- joint r3_shoulder: origin xyz=0.043008 0.000000 0.020580 rpy=0.000000 0.000000 0.000000 -> xyz=0.042992 0.000000 0.000420 rpy=0.000000 0.000000 0.000000
- joint r3_shoulder_servo_joint: origin xyz=0.043008 0.000000 0.020580 rpy=0.000000 0.000000 0.000000 -> xyz=0.042992 0.000000 0.000420 rpy=0.000000 0.000000 0.000000

Commit message: Add shoulder servo slide offsets and update mesh references; replace old shoulder servo meshes

File: hexapod-v2/hexapod-v2.urdf (robot description, URDF)
Before this commit: robot hexapod_v2, 43 links, 42 joints
Links:
- link l1_shoulder_servo: geometry collision mesh filename=./meshes/servo-shoulder-z180-slid-left.stl scale=0.001 0.001 0.001; visual mesh filename=./meshes/servo-shoulder-z180-slid-left.stl scale=0.001 0.001 0.001
- link l2_shoulder_servo: geometry collision mesh filename=./meshes/servo-shoulder-z180-slid-left.stl scale=0.001 0.001 0.001; visual mesh filename=./meshes/servo-shoulder-z180-slid-left.stl scale=0.001 0.001 0.001
- link l3_shoulder_servo: geometry collision mesh filename=./meshes/servo-shoulder-z180-slid-left.stl scale=0.001 0.001 0.001; visual mesh filename=./meshes/servo-shoulder-z180-slid-left.stl scale=0.001 0.001 0.001
- link r1_shoulder_servo: geometry collision mesh filename=./meshes/servo-shoulder-z180-slid-right.stl scale=0.001 0.001 0.001; visual mesh filename=./meshes/servo-shoulder-z180-slid-right.stl scale=0.001 0.001 0.001
- link r2_shoulder_servo: geometry collision mesh filename=./meshes/servo-shoulder-z180-slid-right.stl scale=0.001 0.001 0.001; visual mesh filename=./meshes/servo-shoulder-z180-slid-right.stl scale=0.001 0.001 0.001
- link r3_shoulder_servo: geometry collision mesh filename=./meshes/servo-shoulder-z180-slid-right.stl scale=0.001 0.001 0.001; visual mesh filename=./meshes/servo-shoulder-z180-slid-right.stl scale=0.001 0.001 0.001

Commit message: Add femur shoulder inset and update shoulder joint origins in URDF

File: hexapod-v2/hexapod-v2.urdf (robot description, URDF)
Before this commit: robot hexapod_v2, 43 links, 42 joints
Joints:
- joint l1_shoulder: origin xyz=0.043008 0.000000 0.000420 rpy=0.000000 0.000000 0.000000 -> xyz=0.043008 0.008000 0.000420 rpy=0.000000 0.000000 0.000000
- joint l2_shoulder: origin xyz=0.043008 0.000000 0.000420 rpy=0.000000 0.000000 0.000000 -> xyz=0.043008 0.008000 0.000420 rpy=0.000000 0.000000 0.000000
- joint l3_shoulder: origin xyz=0.043008 0.000000 0.000420 rpy=0.000000 0.000000 0.000000 -> xyz=0.043008 0.008000 0.000420 rpy=0.000000 0.000000 0.000000
- joint r1_shoulder: origin xyz=0.042992 0.000000 0.000420 rpy=0.000000 0.000000 0.000000 -> xyz=0.042992 0.008000 0.000420 rpy=0.000000 0.000000 0.000000
- joint r2_shoulder: origin xyz=0.042992 0.000000 0.000420 rpy=0.000000 0.000000 0.000000 -> xyz=0.042992 0.008000 0.000420 rpy=0.000000 0.000000 0.000000
- joint r3_shoulder: origin xyz=0.042992 0.000000 0.000420 rpy=0.000000 0.000000 0.000000 -> xyz=0.042992 0.008000 0.000420 rpy=0.000000 0.000000 0.000000

Commit message: Update femur shoulder inset and adjust shoulder joint origins for improved alignment

File: hexapod-v2/hexapod-v2.urdf (robot description, URDF)
Before this commit: robot hexapod_v2, 43 links, 42 joints
Joints:
- joint l1_shoulder: origin xyz=0.043008 0.008000 0.000420 rpy=0.000000 0.000000 0.000000 -> xyz=0.043008 0.009000 0.000420 rpy=0.000000 0.000000 0.000000
- joint l2_shoulder: origin xyz=0.043008 0.008000 0.000420 rpy=0.000000 0.000000 0.000000 -> xyz=0.043008 0.009000 0.000420 rpy=0.000000 0.000000 0.000000
- joint l3_shoulder: origin xyz=0.043008 0.008000 0.000420 rpy=0.000000 0.000000 0.000000 -> xyz=0.043008 0.009000 0.000420 rpy=0.000000 0.000000 0.000000
- joint r1_shoulder: origin xyz=0.042992 0.008000 0.000420 rpy=0.000000 0.000000 0.000000 -> xyz=0.042992 0.009000 0.000420 rpy=0.000000 0.000000 0.000000
- joint r2_shoulder: origin xyz=0.042992 0.008000 0.000420 rpy=0.000000 0.000000 0.000000 -> xyz=0.042992 0.009000 0.000420 rpy=0.000000 0.000000 0.000000
- joint r3_shoulder: origin xyz=0.042992 0.008000 0.000420 rpy=0.000000 0.000000 0.000000 -> xyz=0.042992 0.009000 0.000420 rpy=0.000000 0.000000 0.000000

Commit message: Refactor femur shoulder inset to support left and right configurations; adjust URDF joint origins for correct alignment

File: hexapod-v2/hexapod-v2.urdf (robot description, URDF)
Before this commit: robot hexapod_v2, 43 links, 42 joints
Joints:
- joint l1_shoulder: origin xyz=0.043008 0.009000 0.000420 rpy=0.000000 0.000000 0.000000 -> xyz=0.043008 -0.009000 0.000420 rpy=0.000000 0.000000 0.000000
- joint l2_shoulder: origin xyz=0.043008 0.009000 0.000420 rpy=0.000000 0.000000 0.000000 -> xyz=0.043008 -0.009000 0.000420 rpy=0.000000 0.000000 0.000000
- joint l3_shoulder: origin xyz=0.043008 0.009000 0.000420 rpy=0.000000 0.000000 0.000000 -> xyz=0.043008 -0.009000 0.000420 rpy=0.000000 0.000000 0.000000
