Commit message: Update URDF and STL files for knee joint alignment; adjust parent links and origin positions

File: hexapod-v2/hexapod-v2.urdf (robot description, URDF)
Before this commit: robot hexapod_v2, 43 links, 42 joints
Joints:
- joint l1_knee_servo_joint: origin xyz=0.060000 0.000000 0.000000 rpy=0.000000 0.000000 0.000000 -> xyz=0.000000 0.000000 0.000000 rpy=0.000000 0.000000 0.000000; parent l1_femur -> l1_tibia
- joint l1_tip_joint: origin xyz=0.022514 0.004531 -0.095727 rpy=0.000000 0.000000 0.000000 -> xyz=0.022514 -0.004531 -0.095727 rpy=0.000000 0.000000 0.000000
- joint l2_knee_servo_joint: origin xyz=0.060000 0.000000 0.000000 rpy=0.000000 0.000000 0.000000 -> xyz=0.000000 0.000000 0.000000 rpy=0.000000 0.000000 0.000000; parent l2_femur -> l2_tibia
- joint l2_tip_joint: origin xyz=0.022514 0.004531 -0.095727 rpy=0.000000 0.000000 0.000000 -> xyz=0.022514 -0.004531 -0.095727 rpy=0.000000 0.000000 0.000000
- joint l3_knee_servo_joint: origin xyz=0.060000 0.000000 0.000000 rpy=0.000000 0.000000 0.000000 -> xyz=0.000000 0.000000 0.000000 rpy=0.000000 0.000000 0.000000; parent l3_femur -> l3_tibia
- joint l3_tip_joint: origin xyz=0.022514 0.004531 -0.095727 rpy=0.000000 0.000000 0.000000 -> xyz=0.022514 -0.004531 -0.095727 rpy=0.000000 0.000000 0.000000
- joint r1_knee_servo_joint: origin xyz=0.060000 0.000000 0.000000 rpy=0.000000 0.000000 0.000000 -> xyz=0.000000 0.000000 0.000000 rpy=0.000000 0.000000 0.000000; parent r1_femur -> r1_tibia
- joint r1_tip_joint: origin xyz=0.022531 -0.004531 -0.095727 rpy=0.000000 0.000000 0.000000 -> xyz=0.022531 0.004531 -0.095727 rpy=0.000000 0.000000 0.000000
- joint r2_knee_servo_joint: origin xyz=0.060000 0.000000 0.000000 rpy=0.000000 0.000000 0.000000 -> xyz=0.000000 0.000000 0.000000 rpy=0.000000 0.000000 0.000000; parent r2_femur -> r2_tibia
- joint r2_tip_joint: origin xyz=0.022531 -0.004531 -0.095727 rpy=0.000000 0.000000 0.000000 -> xyz=0.022531 0.004531 -0.095727 rpy=0.000000 0.000000 0.000000
- joint r3_knee_servo_joint: origin xyz=0.060000 0.000000 0.000000 rpy=0.000000 0.000000 0.000000 -> xyz=0.000000 0.000000 0.000000 rpy=0.000000 0.000000 0.000000; parent r3_femur -> r3_tibia
- joint r3_tip_joint: origin xyz=0.022531 -0.004531 -0.095727 rpy=0.000000 0.000000 0.000000 -> xyz=0.022531 0.004531 -0.095727 rpy=0.000000 0.000000 0.000000

Commit message: Update tibia joint origins for correct alignment; modify rotation calculations and replace STL files

File: hexapod-v2/hexapod-v2.urdf (robot description, URDF)
Before this commit: robot hexapod_v2, 43 links, 42 joints
Joints:
- joint l1_tip_joint: origin xyz=0.022514 -0.004531 -0.095727 rpy=0.000000 0.000000 0.000000 -> xyz=-0.022531 0.004531 -0.095727 rpy=0.000000 0.000000 0.000000
- joint l2_tip_joint: origin xyz=0.022514 -0.004531 -0.095727 rpy=0.000000 0.000000 0.000000 -> xyz=-0.022531 0.004531 -0.095727 rpy=0.000000 0.000000 0.000000
- joint l3_tip_joint: origin xyz=0.022514 -0.004531 -0.095727 rpy=0.000000 0.000000 0.000000 -> xyz=-0.022531 0.004531 -0.095727 rpy=0.000000 0.000000 0.000000
- joint r1_tip_joint: origin xyz=0.022531 0.004531 -0.095727 rpy=0.000000 0.000000 0.000000 -> xyz=-0.022514 -0.004531 -0.095727 rpy=0.000000 0.000000 0.000000
- joint r2_tip_joint: origin xyz=0.022531 0.004531 -0.095727 rpy=0.000000 0.000000 0.000000 -> xyz=-0.022514 -0.004531 -0.095727 rpy=0.000000 0.000000 0.000000
- joint r3_tip_joint: origin xyz=0.022531 0.004531 -0.095727 rpy=0.000000 0.000000 0.000000 -> xyz=-0.022514 -0.004531 -0.095727 rpy=0.000000 0.000000 0.000000

Commit message: Add knee servo images and update URDF for joint origin adjustments; modify STL files for tibia and knee components

File: hexapod-v2/hexapod-v2.urdf (robot description, URDF)
Before this commit: robot hexapod_v2, 43 links, 42 joints
Joints:
- joint l1_tip_joint: origin xyz=-0.022531 0.004531 -0.095727 rpy=0.000000 0.000000 0.000000 -> xyz=-0.022514 0.004531 -0.115887 rpy=0.000000 0.000000 0.000000
- joint l2_tip_joint: origin xyz=-0.022531 0.004531 -0.095727 rpy=0.000000 0.000000 0.000000 -> xyz=-0.022514 0.004531 -0.115887 rpy=0.000000 0.000000 0.000000
- joint l3_tip_joint: origin xyz=-0.022531 0.004531 -0.095727 rpy=0.000000 0.000000 0.000000 -> xyz=-0.022514 0.004531 -0.115887 rpy=0.000000 0.000000 0.000000
- joint r1_tip_joint: origin xyz=-0.022514 -0.004531 -0.095727 rpy=0.000000 0.000000 0.000000 -> xyz=-0.022531 -0.004531 -0.115887 rpy=0.000000 0.000000 0.000000
- joint r2_tip_joint: origin xyz=-0.022514 -0.004531 -0.095727 rpy=0.000000 0.000000 0.000000 -> xyz=-0.022531 -0.004531 -0.115887 rpy=0.000000 0.000000 0.000000
- joint r3_tip_joint: origin xyz=-0.022514 -0.004531 -0.095727 rpy=0.000000 0.000000 0.000000 -> xyz=-0.022531 -0.004531 -0.115887 rpy=0.000000 0.000000 0.000000

Commit message: Add shoulder mount offsets and adjust URDF joint origins for correct alignment

File: hexapod-v2/hexapod-v2.urdf (robot description, URDF)
Before this commit: robot hexapod_v2, 43 links, 42 joints
Joints:
- joint l1_shoulder: origin xyz=0.043008 -0.009000 0.000420 rpy=0.000000 0.000000 0.000000 -> xyz=0.043008 -0.009000 0.002000 rpy=0.000000 0.000000 0.000000
- joint l1_shoulder_servo_joint: origin xyz=0.043008 0.000000 0.000420 rpy=0.000000 0.000000 0.000000 -> xyz=0.043008 0.000000 0.002000 rpy=0.000000 0.000000 0.000000
- joint l2_shoulder: origin xyz=0.043008 -0.009000 0.000420 rpy=0.000000 0.000000 0.000000 -> xyz=0.043008 -0.009000 0.002000 rpy=0.000000 0.000000 0.000000
- joint l2_shoulder_servo_joint: origin xyz=0.043008 0.000000 0.000420 rpy=0.000000 0.000000 0.000000 -> xyz=0.043008 0.000000 0.002000 rpy=0.000000 0.000000 0.000000
- joint l3_shoulder: origin xyz=0.043008 -0.009000 0.000420 rpy=0.000000 0.000000 0.000000 -> xyz=0.043008 -0.009000 0.002000 rpy=0.000000 0.000000 0.000000
- joint l3_shoulder_servo_joint: origin xyz=0.043008 0.000000 0.000420 rpy=0.000000 0.000000 0.000000 -> xyz=0.043008 0.000000 0.002000 rpy=0.000000 0.000000 0.000000
- joint r1_shoulder: origin xyz=0.042992 0.009000 0.000420 rpy=0.000000 0.000000 0.000000 -> xyz=0.042992 0.009000 0.002000 rpy=0.000000 0.000000 0.000000
- joint r1_shoulder_servo_joint: origin xyz=0.042992 0.000000 0.000420 rpy=0.000000 0.000000 0.000000 -> xyz=0.042992 0.000000 0.002000 rpy=0.000000 0.000000 0.000000
- joint r2_shoulder: origin xyz=0.042992 0.009000 0.000420 rpy=0.000000 0.000000 0.000000 -> xyz=0.042992 0.009000 0.002000 rpy=0.000000 0.000000 0.000000
- joint r2_shoulder_servo_joint: origin xyz=0.042992 0.000000 0.000420 rpy=0.000000 0.000000 0.000000 -> xyz=0.042992 0.000000 0.002000 rpy=0.000000 0.000000 0.000000
- joint r3_shoulder: origin xyz=0.042992 0.009000 0.000420 rpy=0.000000 0.000000 0.000000 -> xyz=0.042992 0.009000 0.002000 rpy=0.000000 0.000000 0.000000
- joint r3_shoulder_servo_joint: origin xyz=0.042992 0.000000 0.000420 rpy=0.000000 0.000000 0.000000 -> xyz=0.042992 0.000000 0.002000 rpy=0.000000 0.000000 0.000000

Commit message: Update tibia slide offsets and adjust joint origins for improved alignment; replace STL files for left and right tibia components

File: hexapod-v2/hexapod-v2.urdf (robot description, URDF)
Before this commit: robot hexapod_v2, 43 links, 42 joints
Joints:
- joint l1_tip_joint: origin xyz=-0.022514 0.004531 -0.115887 rpy=0.000000 0.000000 0.000000 -> xyz=-0.022514 0.010531 -0.115887 rpy=0.000000 0.000000 0.000000
- joint l2_tip_joint: origin xyz=-0.022514 0.004531 -0.115887 rpy=0.000000 0.000000 0.000000 -> xyz=-0.022514 0.010531 -0.115887 rpy=0.000000 0.000000 0.000000
- joint l3_tip_joint: origin xyz=-0.022514 0.004531 -0.115887 rpy=0.000000 0.000000 0.000000 -> xyz=-0.022514 0.010531 -0.115887 rpy=0.000000 0.000000 0.000000
- joint r1_tip_joint: origin xyz=-0.022531 -0.004531 -0.115887 rpy=0.000000 0.000000 0.000000 -> xyz=-0.022531 -0.010531 -0.115887 rpy=0.000000 0.000000 0.000000
- joint r2_tip_joint: origin xyz=-0.022531 -0.004531 -0.115887 rpy=0.000000 0.000000 0.000000 -> xyz=-0.022531 -0.010531 -0.115887 rpy=0.000000 0.000000 0.000000
- joint r3_tip_joint: origin xyz=-0.022531 -0.004531 -0.115887 rpy=0.000000 0.000000 0.000000 -> xyz=-0.022531 -0.010531 -0.115887 rpy=0.000000 0.000000 0.000000
